Commit message: updated dimension to match physical robot

File: src/tomauto1_description/urdf/lidar.xacro (robot description, xacro)
@@ -6,5 +6,5 @@
           <geometry>
               <!-- Example dimensions for a common Lidar -->
-              <cylinder radius="0.05" length="0.04"/>
+              <cylinder radius="0.019" length="0.038"/>
           </geometry>
           <!-- Position the visual relative to the link's origin -->
@@ -30,5 +30,5 @@
       <child link="base_scan"/>
       <!-- Position the lidar on top of the parent link (adjust xyz values as needed) -->
-      <origin xyz="0.215 0 0.225" rpy="0 0 0"/>
+      <origin xyz="0.135 0 0.125" rpy="0 0 0"/>
   </joint>
   <gazebo reference="base_scan">

File: src/tomauto1_description/urdf/mobile_base.xacro (robot description, xacro)
@@ -1,9 +1,9 @@
 <?xml version="1.0"?>
 <robot xmlns:xacro="http://www.ros.org/wiki/xacro">
-    <xacro:property name="base_length" value="0.6" />
-    <xacro:property name="base_width" value="0.4" />
-    <xacro:property name="base_height" value="0.2" />
-    <xacro:property name="wheel_radius" value="0.1" />
-    <xacro:property name="wheel_length" value="0.05" />
+    <xacro:property name="base_length" value="0.336" />
+    <xacro:property name="base_width" value="0.288" />
+    <xacro:property name="base_height" value="0.120" />
+    <xacro:property name="wheel_radius" value="0.06" />
+    <xacro:property name="wheel_length" value="0.032" />
     <link name="base_footprint" />
     <link name="base_link">

Commit message: progress, got the lidar working properly and drifting less, but still not perfect, robot has to be travelling at .1 speed

File: src/tomauto1_description/urdf/lidar.xacro (robot description, xacro)
@@ -10,5 +10,5 @@
           <!-- Position the visual relative to the link's origin -->
           <origin xyz="0 0 0" rpy="0 0 0"/>
-          <material name="grey"/>
+          <!-- <material name="grey"/> -->
       </visual>
       <collision>
@@ -47,11 +47,4 @@
                       <max_angle>3.14</max_angle>
                   </horizontal>
-                  <!-- This does not work correctly -->
-                  <!-- <vertical>
-                      <samples>360</samples>
-                      <resolution>1</resolution>
-                      <min_angle>3.14</min_angle>
-                      <max_angle>3.14</max_angle>
-                  </vertical> -->
               </scan>
               <range>

File: src/tomauto1_description/urdf/mobile_base.xacro (robot description, xacro)
@@ -8,4 +8,9 @@
     <link name="base_footprint" />
     <link name="base_link">
+        <gazebo>
+            <plugin filename="gz_ros2_control-system" name="gz_ros2_control::GazeboSimROS2ControlPlugin">
+                <parameters>$(find tomauto1_bringup)/config/tomauto1_controllers.yaml</parameters>
+            </plugin>
+        </gazebo>
         <visual>
             <geometry>
@@ -38,5 +43,5 @@
             <origin xyz="0 0 0" rpy="0 0 0" />
         </collision>
-        <xacro:cylinder_inertia m="1.0" r="${wheel_radius}" l="${wheel_length}"
+        <xacro:cylinder_inertia m="0.2" r="${wheel_radius}" l="${wheel_length}"
                                 o_xyz="0 0 0" o_rpy="${pi / 2.0} 0 0" />
     </link>
@@ -55,5 +60,5 @@
             <origin xyz="0 0 0" rpy="0 0 0" />
         </collision>
-        <xacro:cylinder_inertia m="1.0" r="${wheel_radius}" l="${wheel_length}"
+        <xacro:cylinder_inertia m="0.2" r="${wheel_radius}" l="${wheel_length}"
                                 o_xyz="0 0 0" o_rpy="${pi / 2.0} 0 0" />
     </link>
@@ -72,5 +77,5 @@
             <origin xyz="0 0 0" rpy="0 0 0" />
         </collision>
-        <xacro:cylinder_inertia m="1.0" r="${wheel_radius}" l="${wheel_length}"
+        <xacro:cylinder_inertia m="0.2" r="${wheel_radius}" l="${wheel_length}"
                                 o_xyz="0 0 0" o_rpy="${pi / 2.0} 0 0" />
     </link>
@@ -89,5 +94,5 @@
             <origin xyz="0 0 0" rpy="0 0 0" />
         </collision>
-        <xacro:cylinder_inertia m="1.0" r="${wheel_radius}" l="${wheel_length}"
+        <xacro:cylinder_inertia m="0.2" r="${wheel_radius}" l="${wheel_length}"
                                 o_xyz="0 0 0" o_rpy="${pi / 2.0} 0 0" />
     </link>

File: src/tomauto1_description/urdf/mobile_base_gazebo.xacro (robot description, xacro)
@@ -13,5 +13,5 @@
             <left_joint>front_left_wheel_joint</left_joint>
             <right_joint>front_right_wheel_joint</right_joint>
-            <wheel_separation>0.314</wheel_separation>
+            <wheel_separation>0.33</wheel_separation>
             <wheel_radius>0.06</wheel_radius>
             <frame_id>odom</frame_id>
